File: _autosave-CZTBoardV3.kicad_pcb (KiCad board)
At the start: 2 copper layers, 80 x 100 mm, 34 parts, among them IC1 LD117AS, IC2 LD117AS, U1 ORBOTECH_OMS40G256, U2 DS90LV031, U3 DS90LV032, X1 W237-102, X2 W237-102, X3 W237-103, X4 W237-102, X5 W237-102

Commit message: new layout
Parts:
- removed C5: C5, CZTBoardV3:C0805K
- removed R5, R7, R8: 0, CZTBoardV3:R1206
- removed the X1 at (105.4, 41.9)
- added C10: 0.0123uF, CZTBoardV3:C0805K, F.Cu at (16.2, 12.5)
- added C11: 0.1uF, CZTBoardV3:C0805K, F.Cu at (7.64, 14.5)
- added C12: 0.1uF, CZTBoardV3:C0805K, F.Cu at (20.9, 0.80)
- added C13: 4.7uF, CZTBoardV3:C0805K, F.Cu at (20.6, 3.81)
- added C14: 4.7uF, CZTBoardV3:C0805K, F.Cu at (14.6, 9.86)
- added C15: 0.1uF, CZTBoardV3:C0805K, F.Cu at (11.9, 13.7)
- added C16: 0.1uF, CZTBoardV3:C0805K, F.Cu at (25.2, 0.80)
- added C17: 4.7uF, CZTBoardV3:C0805K, F.Cu at (18.9, 7.26)
- added C18: 4.7uF, CZTBoardV3:C0805K, F.Cu at (24.9, 3.40)
- added C19: 0.1uF, CZTBoardV3:C0805K, F.Cu at (18.9, 9.86)
- added C20: 0.1uF, CZTBoardV3:C0805K, F.Cu at (14.6, 7.26)
- added C21: 4.7uF, CZTBoardV3:C0805K, F.Cu at (23.2, 6.41)
- added C22: 4.7uF, CZTBoardV3:C0805K, F.Cu at (23.2, 9.01)
- added L1: 40uH, Inductor_SMD:L_1206_3216Metric, F.Cu at (9.62, 10.7)
- added L2: 100uH, Inductor_SMD:L_1206_3216Metric, F.Cu at (9.62, 7.25)
- added L3: 100uH, Inductor_SMD:L_1206_3216Metric, F.Cu at (15.6, 4.24)
- added R20: 470k, CZTBoardV3:R1206, F.Cu at (9.74, 4.02)
- added R21: 10E, CZTBoardV3:R1206, F.Cu at (15.7, 1.01)
- added R22: 10E, CZTBoardV3:R1206, F.Cu at (9.74, 1.01)
- added R23: 10E, CZTBoardV3:R1206, F.Cu at (2.50, 14.7)
- added U4: DHT11, Sensor:Aosong_DHT11_5.5x12.0_P2.54mm, F.Cu at (3.22, 2.66)
Connections:
- U1 pad 25: Net-(U1-Pad25) -> (no net)
- U1 pad 32: /MISO_P -> (no net)
- U2 pad 12: Net-(U2-Pad12) -> (no net)
- U2 pad 5: Net-(U2-Pad5) -> (no net)
- U2 pad 6: Net-(U2-Pad6) -> (no net)
- U2 pad 7: Net-(U2-Pad7) -> (no net)
- U3 pad 1: Net-(U3-Pad1) -> (no net)
- U3 pad 10: Net-(U3-Pad10) -> (no net)
- U3 pad 11: Net-(U3-Pad11) -> (no net)
- U3 pad 2: Net-(U3-Pad2) -> (no net)
- U3 pad 3: Net-(U3-Pad3) -> (no net)
- U3 pad 4: Net-(U3-Pad4) -> (no net)
- U3 pad 5: Net-(U3-Pad5) -> (no net)
- U3 pad 6: Net-(U3-Pad6) -> (no net)
- U3 pad 7: Net-(U3-Pad7) -> (no net)
- U3 pad 9: Net-(U3-Pad9) -> (no net)
- X1 pad 1: GND -> AGND
- X1 pad 2: /CZT_VIN -> /VIN5V
Routing:
- net AGND: track 80.2 -> 303.1 mm, vias 0 -> 8
- net DGND: track 186.6 -> 0.00 mm, vias 7 -> 0
- net GND: track 36.3 -> 0.00 mm, vias 5 -> 4
- net VCC: track 49.2 -> 62.4 mm
- net Net-(IC1-Pad4): track 13.2 -> 0.00 mm
- net /VIN5V: track 0.00 -> 10.1 mm, vias 0 -> 1
- net /CZT_VIN: track 10.1 -> 0.00 mm, vias 1 -> 0
Other:
- board text added: "08/2021 AG"
- board text removed: "MAR 2021 ~HSB"

Commit message: added side panel
Parts:
- added J2: DB9_Male, CZTBoardV3:M09V, F.Cu at (254.3, 139.6)
- added LED1: LED, CZTBoardV3:LED3MM, F.Cu at (273.1, 135.5)
- added R5: 0E, CZTBoardV3:R1206, F.Cu at (163.8, 67.3)
- added S1: TL32PO, CZTBoardV3:TL3XPO, F.Cu at (243.9, 149.6)
- moved C11 138.4 mm to (135.9, 66.6)
- moved C13 138.4 mm to (148.9, 55.9)
- moved C15 138.4 mm to (140.2, 65.8)
- moved C17 138.4 mm to (147.2, 59.3)
- moved C19 138.4 mm to (147.2, 61.9)
- moved L3 138.4 mm to (143.9, 56.3)
- moved R21 138.4 mm to (144.0, 53.1)
- moved R23 138.4 mm to (130.8, 66.8)
- moved U4 138.4 mm to (131.5, 54.7)
- moved C10 138.4 mm to (144.5, 64.5)
- moved C12 138.4 mm to (149.1, 52.9)
- moved C14 138.4 mm to (142.9, 61.9)
- moved C16 138.4 mm to (153.4, 52.9)
- moved C18 138.4 mm to (153.2, 55.5)
- moved C20 138.4 mm to (142.9, 59.3)
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Connections:
- C10 pad 1: (no net) -> /EXT_PICO_600V
- R20 pad 1: (no net) -> /EXT_PICO_GND
- U1 pad 25: (no net) -> Net-(U1-Pad25)
- U1 pad 32: (no net) -> /MISO_P
- U2 pad 12: (no net) -> Net-(U2-Pad12)
- U2 pad 5: (no net) -> Net-(U2-Pad5)
- U2 pad 6: (no net) -> Net-(U2-Pad6)
- U2 pad 7: (no net) -> Net-(U2-Pad7)
- U3 pad 1: (no net) -> Net-(U3-Pad1)
- U3 pad 10: (no net) -> Net-(U3-Pad10)
- U3 pad 11: (no net) -> Net-(U3-Pad11)
- U3 pad 2: (no net) -> Net-(U3-Pad2)
- U3 pad 3: (no net) -> Net-(U3-Pad3)
- U3 pad 4: (no net) -> Net-(U3-Pad4)
- U3 pad 5: (no net) -> Net-(U3-Pad5)
- U3 pad 6: (no net) -> Net-(U3-Pad6)
- U3 pad 7: (no net) -> Net-(U3-Pad7)
- U3 pad 9: (no net) -> Net-(U3-Pad9)
- U4 pad 2: (no net) -> /NC
- U4 pad 3: (no net) -> Net-(U4-Pad3)
- U4 pad 4: (no net) -> AGND
Routing:
- net GND: vias 4 -> 0
- removed copper zone on B.Cu, net GND
