File: _autosave-CZTBoardV3.kicad_pcb (KiCad board)
At the start: 2 copper layers, 96.5 x 94 mm, 52 parts, among them IC1 LD117AS, IC2 LD117AS, U1 ORBOTECH_OMS40G256, U2 DS90LV031, U3 DS90LV032, U4 DHT11, X1 W237-102, X2 W237-102, X3 W237-102, X4 W237-102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

Commit message: nearing completion
Parts:
- moved R20 28.1 mm to (109.8, 142.9), turned to 90 degrees
- moved C10 19.4 mm to (106.0, 142.3), turned to 90 degrees
- moved L1 18.6 mm to (104.7, 116.8), turned to 270 degrees
- moved C21 13.7 mm to (98.3, 130.9)
- moved L2 9.19 mm to (99.5, 123.0)
- moved U4 9.01 mm to (90.0, 122.0)
- moved C15 8.30 mm to (112.4, 134.2), turned to 270 degrees
- moved C14 8.22 mm to (105.0, 123.8)
- moved C17 8.08 mm to (99.9, 138.1), turned to 270 degrees
- moved R23 7.46 mm to (115.7, 132.2), turned to 270 degrees
- moved C20 7.44 mm to (123.9, 130.7)
- moved C19 7.04 mm to (95.9, 135.1), turned to 270 degrees
- moved C18 6.20 mm to (104.2, 135.8), turned to 270 degrees
- moved C11 4.58 mm to (108.1, 134.8), turned to 270 degrees
- moved C12 3.33 mm to (119.6, 130.2), turned to 270 degrees
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Connections:
- C12 pad 1: Net-(C12-Pad1) -> /AVFE_LDO
- C15 pad 1: VDD -> VCC
- C16 pad 1: VDD -> VCC
- C2 pad 1: VDD -> VCC
- C3 pad 1: VDD -> VCC
- C4 pad 1: VDD -> VCC
- L2 pad 1: VDD -> VCC
- L2 pad 2: VDD -> VCC
- R12 pad 1: VDD -> VCC
- R14 pad 2: VDD -> VCC
- R15 pad 2: VDD -> VCC
- R16 pad 2: VDD -> VCC
- R18 pad 2: VDD -> VCC
- R21 pad 1: Net-(C12-Pad1) -> /AVFE_LDO
- R22 pad 1: VDD -> VCC
- R9 pad 2: VDD -> VCC
- U1 pad 39: VDD -> VCC
- U1 pad 40: VDD -> VCC
- U2 pad 16: VDD -> VCC
- U2 pad 4: VDD -> VCC
- U3 pad 16: VDD -> VCC
Routing:
- net AGND: track 333.1 -> 335.9 mm
