File: CZTBoardV3.sch (KiCad schematic (older format))
At the start: 53 parts, among them IC1 LD117AS, IC2 LD117AS, U1 ORBOTECH_OMS40G256, U2 DS90LV031, U3 DS90LV032, U4 DHT11, X1 W237-102, X2 W237-102, X3 W237-103, X4 W237-102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

Commit message: changes to temperature sensor connection
Connections:
- wire segments 183 -> 186
Other:
- moved on the sheet: U4
Changed lines of the file:
@@
 L Sensor:DHT11 U4
 U 1 1 6156F1D7
-P 9350 5800
-F 0 "U4" V 9106 5846 50  0000 R CNN
-F 1 "DHT11" V 9106 5755 50  0000 R CNN
-F 2 "Sensor:Aosong_DHT11_5.5x12.0_P2.54mm" H 9106 5755 50  0001 R CNN
-F 3 "http://akizukidenshi.com/download/ds/aosong/DHT11.pdf" H 9106 5664 50  0001 R CNN
-	1    9350 5800
+P 7775 6275
+F 0 "U4" V 7531 6321 50  0000 R CNN
+F 1 "DHT11" V 7531 6230 50  0000 R CNN
+F 2 "Sensor:Aosong_DHT11_5.5x12.0_P2.54mm" H 7531 6230 50  0001 R CNN
+F 3 "http://akizukidenshi.com/download/ds/aosong/DHT11.pdf" H 7531 6139 50  0001 R CNN
+	1    7775 6275
 	0    -1   -1   0
 $EndComp
+Wire Wire Line
+	7775 5975 7775 5600
+Wire Wire Line
+	8075 6275 8650 6275
+Wire Wire Line
+	7475 6275 7150 6275
+Text Label 7150 6275 0    50   ~ 0
+VCC
 $EndSCHEMATC

Commit message: new layout
Parts:
- removed C8, C9: 0.0123uF, CZTBoardV3:C0805K, symbol Device:CP1
- removed R19: 2m, Resistor_SMD:R_1206_3216Metric, symbol Device:R_US
Connections:
- wire segments 186 -> 174

Commit message: added side panel
Parts:
- added R5: 0E, CZTBoardV3:R1206, symbol CZTBoardV3-eagle-import:R-US_R1206
Connections:
- net labels added: NC
- wire segments 174 -> 178
Other:
- note added: "External Temperature Sensor"
- moved on the sheet: C11, C12, C13, C14, IC2, L1, R21, U4

Commit message: nearing completion
Parts:
- removed L1: 40uH, Inductor_SMD:L_1206_3216Metric, symbol Device:L_Core_Ferrite_Coupled
- removed R5, R6: 0E, CZTBoardV3:R1206, symbol CZTBoardV3-eagle-import:R-US_R1206
- added X1: W237-102, CZTBoardV3:W237-102, symbol CZTBoardV3-eagle-import:W237-102
- renumbered X1 to X3, X5 to X4, X4 to X5, X3 to X6
Connections:
- net labels added: TCK, TDI, TMS
- wire segments 178 -> 163
Other:
- moved on the sheet: R14, R16

Commit message: simplistic design
Parts:
- removed C15, C16, C19, C20: 0.1uF, CZTBoardV3:C0805K, symbol Device:CP1
- removed C17, C18, C21, C22: 4.7uF, CZTBoardV3:C0805K, symbol Device:CP1
- removed L2, L3: 100uH, Inductor_SMD:L_1206_3216Metric, symbol pspice:INDUCTOR
- removed R22, R23: 10E, CZTBoardV3:R1206, symbol Device:R_US
Connections:
- net labels removed: AVDD_LDO, AVFE_LDO, DVDD_LDO
- wire segments 163 -> 128
Other:
- note removed: "LV filtering circuit"
- moved on the sheet: U2, X4A, X4B, X5A
