File: CZTBoardV3.kicad_pcb (KiCad board)
At the start: 2 copper layers, 96.5 x 94 mm, 52 parts, among them IC1 LD117AS, IC2 LD117AS, U1 ORBOTECH_OMS40G256, U2 DS90LV031, U3 DS90LV032, U4 DHT11, X1 W237-102, X2 W237-102, X3 W237-102, X4 W237-102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

Commit message: push
Parts:
- moved U4 96.1 mm to (190.1, 141.1)
- moved R20 25.7 mm to (112.6, 139.4), turned to 90 degrees
- moved L1 18.6 mm to (104.7, 116.8), turned to 270 degrees
- moved C10 17.0 mm to (107.8, 139.6), turned to 90 degrees
- moved C21 13.7 mm to (98.3, 130.9)
- moved C22 12.0 mm to (101.8, 132.2), turned to 270 degrees
- moved L2 10.2 mm to (102.1, 121.5), turned to 270 degrees
- moved C17 9.63 mm to (99.4, 135.1), turned to 270 degrees
- moved C14 9.51 mm to (106.2, 121.8), turned to 270 degrees
- moved C15 8.30 mm to (112.4, 134.2), turned to 270 degrees
- moved R23 7.46 mm to (115.7, 132.2), turned to 270 degrees
- moved C20 7.44 mm to (123.9, 130.7)
- moved C19 7.04 mm to (95.9, 135.1), turned to 270 degrees
- moved C18 6.20 mm to (104.2, 135.8), turned to 270 degrees
- moved C11 4.58 mm to (108.1, 134.8), turned to 270 degrees
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Connections:
- C12 pad 1: Net-(C12-Pad1) -> /AVFE_LDO
- C15 pad 1: VDD -> VCC
- C16 pad 1: VDD -> VCC
- C2 pad 1: VDD -> VCC
- C3 pad 1: VDD -> VCC
- C4 pad 1: VDD -> VCC
- L2 pad 1: VDD -> VCC
- L2 pad 2: VDD -> VCC
- R12 pad 1: VDD -> VCC
- R14 pad 2: VDD -> VCC
- R15 pad 2: VDD -> VCC
- R16 pad 2: VDD -> VCC
- R18 pad 2: VDD -> VCC
- R21 pad 1: Net-(C12-Pad1) -> /AVFE_LDO
- R22 pad 1: VDD -> VCC
- R9 pad 2: VDD -> VCC
- U1 pad 39: VDD -> VCC
- U1 pad 40: VDD -> VCC
- U2 pad 16: VDD -> VCC
- U2 pad 4: VDD -> VCC
- U3 pad 16: VDD -> VCC
Routing:
- net /HV: track 0.00 -> 43.4 mm, vias 0 -> 1
- net AGND: track 333.1 -> 371.7 mm
- net /EXT_PICO_600V: track 0.00 -> 11.6 mm, vias 0 -> 2
- net /EXT_PICO_GND: track 0.00 -> 11.2 mm, vias 0 -> 1
- net VCC: track 62.4 -> 69.1 mm

Commit message: simplistic design
Parts:
- removed C15, C16, C19, C20: 0.1uF, CZTBoardV3:C0805K
- removed C17, C18, C21, C22: 4.7uF, CZTBoardV3:C0805K
- removed L1: 40uH, Inductor_SMD:L_1206_3216Metric
- removed L2, L3: 100uH, Inductor_SMD:L_1206_3216Metric
- removed R22, R23: 10E, CZTBoardV3:R1206
- removed R5, R6: 0E, CZTBoardV3:R1206
- C10, R20: moved to B.Cu
- moved R21 94.2 mm to (205.6, 109.5), turned to 0 degrees
- moved C14 91.1 mm to (197.3, 123.0), turned to 0 degrees
- moved C13 75.4 mm to (177.1, 102.8), turned to 0 degrees
- moved C4 75.3 mm to (212.8, 113.0)
- moved C11 74.0 mm to (177.1, 108.0), turned to 0 degrees
- moved IC2 68.4 mm to (178.9, 86.5), turned to 0 degrees
- moved C12 62.6 mm to (177.1, 105.4), turned to 0 degrees
- moved C6 59.3 mm to (177.1, 110.6), turned to 0 degrees
- moved R14 55.6 mm to (186.2, 118.8)
- moved R16 50.7 mm to (186.2, 121.8)
- moved R3 46.7 mm to (216.9, 109.9), turned to 0 degrees
- moved C2 37.6 mm to (197.3, 118.5), turned to 0 degrees
- moved R4 36.9 mm to (182.4, 130.2), turned to 0 degrees
- moved R15 35.4 mm to (180.2, 121.8)
- moved R1 34.9 mm to (181.5, 126.0), turned to 0 degrees
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Connections:
- C11 pad 1: /AVFE_LDO -> /AVFE
- C12 pad 1: /AVFE_LDO -> /AVFE
- C2 pad 2: AGND -> DGND
- C3 pad 2: AGND -> DGND
- C4 pad 2: AGND -> DGND
- IC2 pad 4: /AVFE_LDO -> /AVFE
- R13 pad 1: AGND -> DGND
- R17 pad 2: AGND -> DGND
- R21 pad 1: /AVFE_LDO -> /AVFE
- U1 pad 21: AGND -> DGND
- U1 pad 22: AGND -> DGND
- U1 pad 35: AGND -> DGND
- U1 pad 36: AGND -> DGND
- U2 pad 8: AGND -> DGND
- U3 pad 12: AGND -> DGND
- U3 pad 8: AGND -> DGND
Routing:
- net AGND: track 371.7 -> 0.00 mm, vias 8 -> 0
- net VDD: track 206.2 -> 0.00 mm, vias 6 -> 0
- net /GPIO: track 138.6 -> 0.00 mm, vias 1 -> 0
- net /RST: track 134.5 -> 0.00 mm, vias 1 -> 0
- net /SS_P: track 119.1 -> 0.00 mm, vias 2 -> 0
- net /PWR_ON: track 113.0 -> 0.00 mm, vias 1 -> 0
- net /MISO_P: track 96.9 -> 0.00 mm, vias 2 -> 0
- net /MISO: track 76.0 -> 0.00 mm, vias 1 -> 0
- net /MOSI_P: track 71.3 -> 0.00 mm, vias 2 -> 0
- net /SS_N: track 70.1 -> 0.00 mm
- net VCC: track 69.1 -> 0.00 mm
- net /MOSI_N: track 57.0 -> 0.00 mm
- net /MISO_N: track 51.3 -> 0.00 mm, vias 2 -> 0
- net /CLK_P: track 44.5 -> 0.00 mm, vias 2 -> 0
- net /AVFE: track 41.6 -> 0.00 mm
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Other:
- board size 96.5 x 94 mm -> 7 x 11 mm
- board text removed: "08/2021 AG"

Commit message: half routing done
Parts:
- moved R17 60.6 mm to (233.7, 76.2), turned to 90 degrees
- moved U4 58.9 mm to (185.4, 72.4), turned to 90 degrees
- moved R13 54.3 mm to (231.0, 99.7), turned to 270 degrees
- moved R18 49.9 mm to (142.5, 123.2), turned to 90 degrees
- moved R1 49.6 mm to (228.6, 110.5), turned to 90 degrees
- moved C4 45.1 mm to (167.7, 113.4), turned to 270 degrees
- moved R9 44.9 mm to (160.8, 108.0), turned to 270 degrees
- moved U2 37.7 mm to (198.0, 84.8)
- moved R4 37.6 mm to (145.4, 123.1), turned to 270 degrees
- moved R12 36.8 mm to (169.2, 108.0), turned to 90 degrees
- moved IC2 35.0 mm to (171.4, 120.7)
- moved C2 33.3 mm to (171.0, 98.1), turned to 270 degrees
- moved R21 29.7 mm to (176.5, 115.1), turned to 90 degrees
- moved C14 28.2 mm to (176.5, 103.9), turned to 90 degrees
- moved R15 26.5 mm to (157.5, 108.1), turned to 270 degrees
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Routing:
- net AGND: track 0.00 -> 108.3 mm, vias 0 -> 1
- net VCC: track 0.00 -> 101.0 mm
- net /PWR_ON: track 0.00 -> 66.9 mm, vias 0 -> 1
- net /SS_P: track 0.00 -> 52.2 mm
- net /CLK: track 47.8 -> 0.00 mm, vias 1 -> 0
- net /TCK: track 0.00 -> 46.8 mm
- net /MOSI: track 44.3 -> 0.00 mm, vias 1 -> 0
- net /TDI: track 0.00 -> 40.4 mm
- net /SS: track 38.7 -> 0.00 mm, vias 1 -> 0
- net /RST: track 0.00 -> 22.5 mm
- net /AVFE: track 0.00 -> 20.8 mm
- net /TMS: track 0.00 -> 18.9 mm
- net Net-(C13-Pad1): track 0.00 -> 4.11 mm
- net DGND: track 0.00 -> 3.08 mm
- net /MISO_P: track 0.00 -> 2.98 mm
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
Commit message: layout done
Parts:
- added REF**: MountingHole_3.2mm_M3, MountingHole:MountingHole_3.2mm_M3, F.Cu at (209.7, 146.1)
- added REF**: MountingHole_3.2mm_M3, MountingHole:MountingHole_3.2mm_M3, F.Cu at (111.7, 75.3)
- added REF**: MountingHole_3.2mm_M3, MountingHole:MountingHole_3.2mm_M3, F.Cu at (112.3, 146.3)
- added REF**: MountingHole_3.2mm_M3, MountingHole:MountingHole_3.2mm_M3, F.Cu at (210.3, 75.7)
- moved R1 72.8 mm to (159.3, 88.2)
- moved R17 61.5 mm to (197.7, 126.1), turned to 270 degrees
- moved R13 56.8 mm to (174.7, 107.8)
- moved U3 46.0 mm to (191.5, 123.8)
- moved U2 33.3 mm to (164.7, 86.2)
- moved R3 29.0 mm to (171.4, 85.2)
- moved R2 28.8 mm to (171.9, 107.8), turned to 270 degrees
- moved U4 18.9 mm to (181.3, 90.8), turned to 0 degrees
- moved C2 16.3 mm to (165.3, 113.4)
- moved C11 4.09 mm to (186.1, 114.8)
- moved C12 4.09 mm to (183.3, 114.9)
- moved C13 4.09 mm to (180.6, 108.6)
- moved C14 4.09 mm to (180.6, 103.9)
- moved C6 4.09 mm to (188.8, 114.9)
- moved R21 4.09 mm to (180.6, 115.1)
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Routing:
- net VCC: track 101.0 -> 267.8 mm, vias 0 -> 5
- net DGND: track 3.08 -> 169.7 mm, vias 0 -> 4
- net /MOSI: track 0.00 -> 125.7 mm, vias 0 -> 1
- net /CLK: track 0.00 -> 108.5 mm, vias 0 -> 1
- net /MISO_P: track 2.98 -> 108.9 mm, vias 0 -> 3
- net /AVFE: track 20.8 -> 119.5 mm
- net /SS: track 0.00 -> 97.9 mm, vias 0 -> 3
- net /MISO_N: track 0.00 -> 94.5 mm, vias 0 -> 3
- net AGND: track 108.3 -> 197.6 mm, vias 1 -> 4
- net /PWR_ON: track 66.9 -> 155.1 mm
- net /RST: track 22.5 -> 102.9 mm, vias 0 -> 3
- net /MOSI_P: track 0.00 -> 72.8 mm, vias 0 -> 2
- net /CLK_P: track 0.00 -> 67.0 mm
- net /SS_N: track 0.00 -> 62.2 mm, vias 0 -> 4
- net /MOSI_N: track 0.00 -> 61.2 mm, vias 0 -> 2
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Other:
- board size 7 x 11 mm -> 105.6 x 79.1 mm
- board text added: "08/2021 AG"
- board text added: "CZT Interface Card"

Commit message: gerbers included
Parts:
- removed the REF** at (209.7, 146.1)
- removed the REF** at (111.7, 75.3)
- removed the REF** at (112.3, 146.3)
- removed the REF** at (210.3, 75.7)
- added REF**: MountingHole_3.2mm_M3, MountingHole:MountingHole_3.2mm_M3, F.Cu at (203.0, 70.7)
- added REF**: MountingHole_3.2mm_M3, MountingHole:MountingHole_3.2mm_M3, F.Cu at (117.0, 154.4)
- added REF**: MountingHole_3.2mm_M3, MountingHole:MountingHole_3.2mm_M3, F.Cu at (202.6, 154.6)
- added REF**: MountingHole_3.2mm_M3, MountingHole:MountingHole_3.2mm_M3, F.Cu at (117.1, 69.8)
Other:
- board size 105.6 x 79.1 mm -> 95.8 x 93.2 mm
Changed lines of the file:
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@@
   )
   (setup
-    (last_trace_width 0.6096)
+    (last_trace_width 0.25)
     (user_trace_width 0.6096)
     (trace_clearance 0.1524)
@@
       (padsonsilk false)
       (subtractmaskfromsilk false)
-      (outputformat 5)
+      (outputformat 4)
       (mirror false)
       (drillshape 2)
       (scaleselection 1)
-      (outputdirectory "svg"))
+      (outputdirectory "pdf"))
   )
   (net 0 "")
@@
   )
   (module MountingHole:MountingHole_3.2mm_M3 (layer Top)
-    (at 209.67 146.11)
+    (at 203.03 70.66)
     (descr "Mounting Hole 3.2mm, no annular, M3")
     (tags "mounting hole 3.2mm no annular m3")
@@
   )
   (module MountingHole:MountingHole_3.2mm_M3 (layer Top)
-    (at 111.68 75.26)
+    (at 116.95 154.38)
     (descr "Mounting Hole 3.2mm, no annular, M3")
     (tags "mounting hole 3.2mm no annular m3")
@@
   )
   (module MountingHole:MountingHole_3.2mm_M3 (layer Top)
-    (at 112.35 146.32)
+    (at 202.62 154.62)
     (descr "Mounting Hole 3.2mm, no annular, M3")
     (tags "mounting hole 3.2mm no annular m3")
@@
   )
   (module MountingHole:MountingHole_3.2mm_M3 (layer Top)
-    (at 210.28 75.67)
+    (at 117.11 69.76)
     (descr "Mounting Hole 3.2mm, no annular, M3")
     (tags "mounting hole 3.2mm no annular m3")
@@
       (effects (font (size 1 1) (thickness 0.15)))
     )
-    (fp_text user %R (at 0.3 0) (layer F.Fab)
-      (effects (font (size 1 1) (thickness 0.15)))
-    )
     (fp_circle (center 0 0) (end 3.2 0) (layer Cmts.User) (width 0.15))
     (fp_circle (center 0 0) (end 3.45 0) (layer F.CrtYd) (width 0.05))
+    (fp_text user %R (at 0.3 0) (layer F.Fab)
+      (effects (font (size 1 1) (thickness 0.15)))
+    )
     (pad 1 np_thru_hole circle (at 0 0) (size 3.2 3.2) (drill 3.2) (layers *.Cu *.Mask))
   )
@@
       (net 2 VCC) (solder_mask_margin 0.1016))
   )
+  (dimension 95.640151 (width 0.15) (layer Dwgs.User)
+    (gr_text "95.640 mm" (at 160.082311 161.764998 0.1018430809) (layer Dwgs.User)
+      (effects (font (size 1 1) (thickness 0.15)))
+    )
+    (feature1 (pts (xy 207.9 160.38) (xy 207.901042 160.96642)))
+    (feature2 (pts (xy 112.26 160.55) (xy 112.261042 161.13642)))
+    (crossbar (pts (xy 112.26 160.55) (xy 207.9 160.38)))
+    (arrow1a (pts (xy 207.9 160.38) (xy 206.77454 160.968422)))
+    (arrow1b (pts (xy 207.9 160.38) (xy 206.772456 159.795583)))
+    (arrow2a (pts (xy 112.26 160.55) (xy 113.387544 161.134417)))
+    (arrow2b (pts (xy 112.26 160.55) (xy 113.38546 159.961578)))
+  )
+  (dimension 93.280001 (width 0.15) (layer Dwgs.User)
+    (gr_text "93.280 mm" (at 108.965001 112.69014 270.0061423) (layer Dwgs.User)
+      (effects (font (size 1 1) (thickness 0.15)))
+    )
+    (feature1 (pts (xy 110.28 159.33) (xy 109.68358 159.330064)))
+    (feature2 (pts (xy 110.27 66.05) (xy 109.67358 66.050064)))
+    (crossbar (pts (xy 110.260001 66.050001) (xy 110.270001 159.330001)))
+    (arrow1a (pts (xy 110.270001 159.330001) (xy 109.683459 158.20356)))
+    (arrow1b (pts (xy 110.270001 159.330001) (xy 110.856301 158.203434)))
+    (arrow2a (pts (xy 110.260001 66.050001) (xy 109.673701 67.176568)))
+    (arrow2b (pts (xy 110.260001 66.050001) (xy 110.846543 67.176442)))
+  )
+  (gr_line (start 112.37 66.15) (end 208.06 66.65) (layer Edge.Cuts) (width 0.1))
+  (gr_line (start 112.29 159.3) (end 112.37 66.15) (layer Edge.Cuts) (width 0.1))
+  (gr_line (start 207.86 159.36) (end 112.29 159.3) (layer Edge.Cuts) (width 0.1))
+  (gr_line (start 208.06 66.65) (end 207.86 159.36) (layer Edge.Cuts) (width 0.1))
   (gr_text "CZT Interface Card" (at 193.73 80.05) (layer Top)
     (effects (font (size 1.5 1.5) (thickness 0.3)))
@@
     (effects (font (size 1.5 1.5) (thickness 0.3)) (justify mirror))
   )
-  (dimension 78.970063 (width 0.15) (layer Dwgs.User)
-    (gr_text "78.970 mm" (at 101.799976 110.963139 89.92744618) (layer Dwgs.User)
-      (effects (font (size 1 1) (thickness 0.15)))
-    )
-    (feature1 (pts (xy 103.32 71.48) (xy 102.563555 71.479042)))
-    (feature2 (pts (xy 103.22 150.45) (xy 102.463555 150.449042)))
-    (crossbar (pts (xy 103.049975 150.449785) (xy 103.149975 71.479785)))
-    (arrow1a (pts (xy 103.149975 71.479785) (xy 103.734969 72.60703)))
-    (arrow1b (pts (xy 103.149975 71.479785) (xy 102.562128 72.605545)))
-    (arrow2a (pts (xy 103.049975 150.449785) (xy 103.637822 149.324025)))
-    (arrow2b (pts (xy 103.049975 150.449785) (xy 102.464981 149.32254)))
-  )
-  (dimension 105.09 (width 0.15) (layer Dwgs.User)
-    (gr_text "105.090 mm" (at 160.775 153.11) (layer Dwgs.User)
-      (effects (font (size 1 1) (thickness 0.15)))
-    )
-    (feature1 (pts (xy 213.32 154.46) (xy 213.32 153.823579)))
-    (feature2 (pts (xy 108.23 154.46) (xy 108.23 153.823579)))
-    (crossbar (pts (xy 108.23 154.41) (xy 213.32 154.41)))
-    (arrow1a (pts (xy 213.32 154.41) (xy 212.193496 154.996421)))
-    (arrow1b (pts (xy 213.32 154.41) (xy 212.193496 153.823579)))
-    (arrow2a (pts (xy 108.23 154.41) (xy 109.356504 154.996421)))
-    (arrow2b (pts (xy 108.23 154.41) (xy 109.356504 153.823579)))
-  )
-  (gr_line (start 108.01 71.59) (end 213.54 71.63) (layer Edge.Cuts) (width 0.1))
-  (gr_line (start 108.17 150.68) (end 108.01 71.59) (layer Edge.Cuts) (width 0.1))
-  (gr_line (start 213.59 150.69) (end 108.17 150.68) (layer Edge.Cuts) (width 0.1))
-  (gr_line (start 213.54 71.63) (end 213.59 150.69) (layer Edge.Cuts) (width 0.1))
   (segment (start 155.89 143.52) (end 155.89 129.86) (width 0.6096) (layer Bottom) (net 1))
   (via (at 157.48 128.27) (size 2) (drill 1) (layers Top Bottom) (net 1))
