File: CZTBoardV3.kicad_pcb (KiCad board)
At the start: 2 copper layers, 95.8 x 93.2 mm, 41 parts, among them IC1 LD117AS, IC2 LD117AS, U1 ORBOTECH_OMS40G256, U2 DS90LV031, U3 DS90LV032, U4 DHT11, X1 W237-102, X2 W237-102, X3 W237-102, X4 W237-102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

Commit message: final gerbers with drill files generated as well
Parts:
- C11, C12, C13, C14, C2, C3, C4, C6: footprint Capacitor_THT:C_Rect_L7.2mm_W4.5mm_P5.00mm_FKS2_FKP2_MKS2_MKP2 -> CZTBoardV3:C0805K
- moved C10 0.22 mm to (125.8, 130.1)

Commit message: some changes from pcbpower
Routing:
- net /TDI: track 42.9 -> 41.4 mm
